Commit message: update camera

File: kortex_description/arms/gen3/7dof/urdf/gen3_macro.xacro (robot description, xacro)
@@ -3,4 +3,6 @@
   <!-- Propagate last link name information because it is the gripper's parent link -->
   <xacro:property name="last_arm_link" value="end_effector_link"/>
+  <!-- Include the task_board xacro file -->
+  <!-- <xacro:include filename="$(find robothon_2023_board_description)/urdf/task_board.urdf.xacro"/> -->
   <xacro:macro name="load_arm" params="parent:='' dof vision prefix *origin">
       <link name="${prefix}base_link">
@@ -313,5 +315,5 @@
       <link name="${prefix}camera_link" />
       <joint name="${prefix}camera_module" type="fixed">
-        <origin xyz="0 0.05639 -0.00305" rpy="3.14159265358979 3.14159265358979 0" />
+        <origin xyz="0 0.05639 -0.00305" rpy="-1.57 -1.57 0" />
         <parent link="${prefix}end_effector_link" />
         <child  link="${prefix}camera_link" />
@@ -319,5 +321,5 @@
       <link name="${prefix}camera_depth_frame" />
       <joint name="${prefix}depth_module" type="fixed">
-        <origin xyz="0.0275 0.066 -0.00305" rpy="3.14159265358979 3.14159265358979 0" />
+        <origin xyz="0.0275 0.066 -0.00305" rpy="-1.57 -1.57 0" />
         <parent link="${prefix}end_effector_link" />
         <child  link="${prefix}camera_depth_frame" />
@@ -325,9 +327,40 @@
       <link name="${prefix}camera_color_frame" />
       <joint name="${prefix}color_module" type="fixed">
-        <origin xyz="0 0.05639 -0.00305" rpy="3.14159265358979 3.14159265358979 0" />
+        <origin xyz="0 0.05639 -0.00305" rpy="-1.57 -1.57 0" />
         <parent link="${prefix}end_effector_link" />
         <child  link="${prefix}camera_color_frame" />
       </joint>
     </xacro:if>
+    <gazebo reference="${prefix}camera_link">
+      <sensor type="camera" name="camera_sensor">
+        <camera>
+          <horizontal_fov>1.3962634</horizontal_fov>
+          <image>
+            <width>640</width>
+            <height>480</height>
+            <format>R8G8B8</format>
+          </image>
+          <clip>
+            <near>0.1</near>
+            <far>100</far>
+          </clip>
+        </camera>
+        <plugin name="camera_controller" filename="libgazebo_ros_camera.so">
+          <alwaysOn>true</alwaysOn>
+          <updateRate>30</updateRate>
+          <cameraName>camera</cameraName>
+          <imageTopicName>image_raw</imageTopicName>
+          <cameraInfoTopicName>camera_info</cameraInfoTopicName>
+          <frameName>$(arg color_frame_id)</frameName>
+        </plugin>
+      </sensor>
+    </gazebo>
+    <!-- Add the task board -->
+    <!-- <xacro:task_board board_id="task_board" height="0.085"/>
+    <joint name="task_board_to_world" type="fixed">
+        <parent link="world"/>
+        <child link="task_board_base_link"/>
+        <origin xyz="5 0 0" rpy="0 0 0"/>
+    </joint> -->
   </xacro:macro>
 </robot>

File: kortex_description/robots/gen3.xacro (robot description, xacro)
@@ -8,5 +8,16 @@
     <xacro:arg name="sim" default="false" />
     <xacro:arg name="prefix" default="" />
+    <xacro:arg name="board_id" default="task_board"/>
+    <!-- Load the robot -->
     <xacro:include filename="$(find kortex_description)/robots/kortex_robot.xacro" />
     <xacro:load_robot arm="$(arg arm)" gripper="$(arg gripper)" dof="$(arg dof)" vision="$(arg vision)" sim="$(arg sim)" prefix="$(arg prefix)" />
+    <!-- Load the task board -->
+    <!-- <xacro:include filename="$(find robothon_2023_board_description)/urdf/task_board.urdf.xacro"/>
+    <xacro:task_board board_id="$(arg board_id)" height="0.085"/> -->
+    <!-- Connect the task board to the world -->
+    <!-- <joint name="$(arg board_id)_to_world" type="fixed">
+        <parent link="$(arg prefix)base_link"/>
+        <child link="$(arg board_id)_base_link"/>
+        <origin xyz="1 0 0" rpy="0 0 0"/>
+    </joint> -->
 </robot>

File: kortex_description/robots/gen3_robotiq_2f_85.xacro (robot description, xacro)
@@ -10,3 +10,11 @@
     <xacro:include filename="$(find kortex_description)/robots/kortex_robot.xacro" />
     <xacro:load_robot arm="$(arg arm)" gripper="$(arg gripper)" dof="$(arg dof)" vision="$(arg vision)" sim="$(arg sim)" prefix="$(arg prefix)" />
+    <!-- <xacro:include filename="$(find robothon_2023_board_description)/urdf/task_board.urdf.xacro"/> -->
+    <!-- <xacro:task_board board_id="$(arg board_id)" height="0.085"/> -->
+    <!-- Connect the task board to the world -->
+    <!-- <joint name="$(arg board_id)_to_world" type="fixed">
+        <parent link="$(arg prefix)base_link"/>
+        <child link="$(arg board_id)_base_link"/>
+        <origin xyz="1 0 0" rpy="0 0 0"/>
+    </joint> -->
 </robot>
